Commit message: v1.1: parts list from 23.10.2026, fit check, new logo, fixed rear cover
- 3D viewer: electronics per the new parts list (Pi 3B, PCA9685 + cap,
  MPU-6050, Pi Camera v2, LiPo 2S, XT60, fuse, switch, UBEC, buzzer,
  USB mic/speaker, ADS1115 option); servos seated per bracket STLs
- Built-in fit check: parts vs body and each other, wires through walls,
  servo cable and camera ribbon lengths, camera view, electrical calc
- New Ala-Too IT & Business College logo on the top cover
- Rear cover: K.D.Y engraving filled in the STL, raised ALA-TOO text
- print/: camera mount and rear cover; tools/mounts, tools/logo generators
- CHANGELOG.md with v1.0 and v1.1

File: 3d-viewer/spot_micro.urdf (robot description, URDF)
Before this commit: robot spot_micro_rviz, 24 links, 23 joints
Links:
- link rear_link: geometry collision box size=0.04 0.11 0.07; visual mesh filename=stl/backpart_filled.stl scale=0.001 0.001 0.001

Commit message: v1.2: real KDY0523 print parts in the 3D model
- The mike4192 URDF meshes turned out to be KDY0523 `_mg` parts plus
  servo bodies (ICP match 0.002 mm); the model now uses the parts we
  actually print: `_cls` (PDI-HV5523MG), non-mega covers and side plate,
  mike4192 plain plate
- print/kdy: STLs from Thingiverse 3445283, 4591999, 4596267 (CC BY)
- tools/kdy/fit_kdy.py: part registration and servo seat extraction
- Rear cover: ALA-TOO text is now on R_cover only; the old
  backpart_alatoo.stl fused the bottom and rear covers into one body

File: 3d-viewer/spot_micro.urdf (robot description, URDF)
Before this commit: robot spot_micro_rviz, 24 links, 23 joints
Links:
- link base_link: geometry collision box size=0.14 0.11 0.07; visual mesh filename=stl/kdy/mainbody.stl scale=0.001 0.001 0.001
- link front_left_foot_link: geometry collision box size=0.026 0.020 0.13; visual mesh filename=stl/kdy/lfoot.stl scale=0.001 0.001 0.001
- link front_left_leg_link: geometry collision box size=0.028 0.036 0.1075; visual mesh filename=stl/kdy/larm.stl scale=0.001 0.001 0.001
- link front_left_leg_link_cover: geometry visual mesh filename=stl/kdy/larm_cover.stl scale=0.001 0.001 0.001
- link front_left_shoulder_link: geometry collision box size=0.044 0.038 0.07; visual mesh filename=stl/kdy/lshoulder.stl scale=0.001 0.001 0.001
- link front_link: geometry collision box size=0.058 0.11 0.07; visual mesh filename=stl/kdy/frontpart.stl scale=0.001 0.001 0.001
- link front_right_foot_link: geometry collision box size=0.026 0.020 0.13; visual mesh filename=stl/kdy/rfoot.stl scale=0.001 0.001 0.001
- link front_right_leg_link: geometry collision box size=0.028 0.036 0.1075; visual mesh filename=stl/kdy/rarm.stl scale=0.001 0.001 0.001
- link front_right_leg_link_cover: geometry visual mesh filename=stl/kdy/rarm_cover.stl scale=0.001 0.001 0.001
- link front_right_shoulder_link: geometry collision box size=0.044 0.038 0.07; visual mesh filename=stl/kdy/rshoulder.stl scale=0.001 0.001 0.001
- link rear_left_foot_link: geometry collision box size=0.026 0.020 0.13; visual mesh filename=stl/kdy/lfoot.stl scale=0.001 0.001 0.001
- link rear_left_leg_link: geometry collision box size=0.028 0.036 0.1075; visual mesh filename=stl/kdy/larm.stl scale=0.001 0.001 0.001
- link rear_left_leg_link_cover: geometry visual mesh filename=stl/kdy/larm_cover.stl scale=0.001 0.001 0.001
- link rear_left_shoulder_link: geometry collision box size=0.044 0.038 0.07; visual mesh filename=stl/kdy/lshoulder.stl scale=0.001 0.001 0.001
- link rear_link: geometry collision box size=0.04 0.11 0.07; visual mesh filename=stl/kdy/backpart_alatoo.stl scale=0.001 0.001 0.001
- link rear_right_foot_link: geometry collision box size=0.026 0.020 0.13; visual mesh filename=stl/kdy/rfoot.stl scale=0.001 0.001 0.001
- link rear_right_leg_link: geometry collision box size=0.028 0.036 0.1075; visual mesh filename=stl/kdy/rarm.stl scale=0.001 0.001 0.001
- link rear_right_leg_link_cover: geometry visual mesh filename=stl/kdy/rarm_cover.stl scale=0.001 0.001 0.001
- link rear_right_shoulder_link: geometry collision box size=0.044 0.038 0.07; visual mesh filename=stl/kdy/rshoulder.stl scale=0.001 0.001 0.001
